Commit message: added agv_house.launch

File: my_agv/urdf/my_agv.urdf_v1.xacro (robot description, xacro)
@@ -15,5 +15,5 @@
     <inertial>
       <origin
-        xyz="0.000205357488381168 -0.000114087493545172 0.154772210158345"
+        xyz="0.000205357488381168 -0.000114087493545167 0.154772210158345"
         rpy="0 0 0" />
       <mass
@@ -21,6 +21,6 @@
       <inertia
         ixx="6.3929434908259"
-        ixy="0.00883169715336634"
-        ixz="-0.00530948836048059"
+        ixy="0.00883169715336637"
+        ixz="-0.0053094883604806"
         iyy="15.5817880289174"
         iyz="0.00294971575582209"
@@ -52,8 +52,61 @@
   </link>
   <link
+    name="wheel_right_link">
+    <inertial>
+      <origin
+        xyz="-1.94908591625968E-18 -7.34092456632638E-16 0.0500000000000003"
+        rpy="0 0 0" />
+      <mass
+        value="3.14159265358979" />
+      <inertia
+        ixx="0.010471975511966"
+        ixy="7.08713124779409E-34"
+        ixz="4.70197740328895E-35"
+        iyy="0.010471975511966"
+        iyz="-3.74856813205645E-18"
+        izz="0.015707963267949" />
+    </inertial>
+    <visual>
+      <origin
+        xyz="0 0 0"
+        rpy="0 0 0" />
+      <geometry>
+        <mesh
+          filename="package://my_agv/meshes/wheel_right_link.STL" />
+      </geometry>
+      <material
+        name="">
+        <color
+          rgba="0.792156862745098 0.819607843137255 0.933333333333333 1" />
+      </material>
+    </visual>
+    <collision>
+      <origin
+        xyz="0 0 0"
+        rpy="0 0 0" />
+      <geometry>
+        <mesh
+          filename="package://my_agv/meshes/wheel_right_link.STL" />
+      </geometry>
+    </collision>
+  </link>
+  <joint
+    name="wheel_right_joint"
+    type="continuous">
+    <origin
+      xyz="0 -0.2 0"
+      rpy="1.5708 0 0" />
+    <parent
+      link="base_link" />
+    <child
+      link="wheel_right_link" />
+    <axis
+      xyz="0 0 1" />
+  </joint>
+  <link
     name="wheel_left_link">
     <inertial>
       <origin
-        xyz="-1.94908591625972E-18 -2.06349949181977E-15 0.050000000000001"
+        xyz="-1.94908591625968E-18 7.34092456632637E-16 -0.0500000000000003"
         rpy="0 0 0" />
       <mass
@@ -61,8 +114,8 @@
       <inertia
         ixx="0.010471975511966"
-        ixy="-2.50467333359635E-33"
-        ixz="2.78074600412331E-47"
+        ixy="5.32443059626186E-35"
+        ixz="4.70197740328914E-35"
         iyy="0.010471975511966"
-        iyz="3.28708101219996E-18"
+        iyz="-3.74856813205645E-18"
         izz="0.015707963267949" />
     </inertial>
@@ -96,62 +149,9 @@
     <origin
       xyz="0 0.2 0"
-      rpy="-1.5708 0 0" />
+      rpy="1.5708 0 0" />
     <parent
       link="base_link" />
     <child
       link="wheel_left_link" />
-    <axis
-      xyz="0 0 1" />
-  </joint>
-  <link
-    name="wheel_right_link">
-    <inertial>
-      <origin
-        xyz="-1.94908591626003E-18 2.06349949181977E-15 -0.050000000000001"
-        rpy="0 0 0" />
-      <mass
-        value="3.14159265358979" />
-      <inertia
-        ixx="0.010471975511966"
-        ixy="5.67475236929744E-35"
-        ixz="-6.30024073944018E-49"
-        iyy="0.010471975511966"
-        iyz="3.28708101219996E-18"
-        izz="0.015707963267949" />
-    </inertial>
-    <visual>
-      <origin
-        xyz="0 0 0"
-        rpy="0 0 0" />
-      <geometry>
-        <mesh
-          filename="package://my_agv/meshes/wheel_right_link.STL" />
-      </geometry>
-      <material
-        name="">
-        <color
-          rgba="0.792156862745098 0.819607843137255 0.933333333333333 1" />
-      </material>
-    </visual>
-    <collision>
-      <origin
-        xyz="0 0 0"
-        rpy="0 0 0" />
-      <geometry>
-        <mesh
-          filename="package://my_agv/meshes/wheel_right_link.STL" />
-      </geometry>
-    </collision>
-  </link>
-  <joint
-    name="wheel_right_joint"
-    type="continuous">
-    <origin
-      xyz="0 -0.2 0"
-      rpy="-1.5708 0 0" />
-    <parent
-      link="base_link" />
-    <child
-      link="wheel_right_link" />
     <axis
       xyz="0 0 1" />
@@ -267,5 +267,5 @@
     <inertial>
       <origin
-        xyz="5.55111512312578E-17 0 0.05"
+        xyz="-5.55111512312578E-17 -5.55111512312578E-17 0.05"
         rpy="0 0 0" />
       <mass
@@ -274,5 +274,5 @@
         ixx="0.00114537232162128"
         ixy="3.74939945665464E-36"
-        ixz="-5.87747175411144E-36"
+        ixz="-4.70197740328915E-36"
         iyy="0.00114537232162128"
         iyz="-3.7943922501345E-36"
@@ -314,5 +314,5 @@
       link="base_scan" />
     <axis
-      xyz="0 0 1" />
+      xyz="0 0 0" />
   </joint>
 </robot>
